File: connectors.sch (KiCad schematic (older format))
At the start: 15 parts, among them J1 Conn_ARM_JTAG_SWD_10, J2 47346-0001, J3 Conn_01x04_Male, J4 Conn_01x04_Male, J5 Conn_01x04_Male, J6 Conn_01x04_Male, J7 Conn_01x04_Male, J8 Conn_01x04_Male, U6 USBLC6-2SC6

Commit message: update
Parts:
- added J9: Screw_Terminal_01x02, TerminalBlock_Phoenix:TerminalBlock_Phoenix_MKDS-3-2-5.08_1x02_P5.08mm_Horizontal, symbol Connector:Screw_Terminal_01x02
Connections:
- net GND: now also J9.1 (Pin_1)
- new net VCC: J9.2 (Pin_2)
Changed lines of the file:
@@
 Wire Notes Line
 	3800 2350 7500 2350
+Wire Wire Line
+	4100 3550 4200 3550
+$Comp
+L power:GND #PWR024
+U 1 1 61811988
+P 4200 3800
+F 0 "#PWR024" H 4200 3550 50  0001 C CNN
+F 1 "GND" H 4350 3750 50  0000 C CNN
+F 2 "" H 4200 3800 50  0001 C CNN
+F 3 "" H 4200 3800 50  0001 C CNN
+	1    4200 3800
+	1    0    0    -1
+$EndComp
+Wire Wire Line
+	4200 3650 4100 3650
+$Comp
+L power:VCC #PWR021
+U 1 1 618127F9
+P 4200 3400
+F 0 "#PWR021" H 4200 3250 50  0001 C CNN
+F 1 "VCC" H 4215 3573 50  0000 C CNN
+F 2 "" H 4200 3400 50  0001 C CNN
+F 3 "" H 4200 3400 50  0001 C CNN
+	1    4200 3400
+	1    0    0    -1
+$EndComp
+$Comp
+L Connector:Screw_Terminal_01x02 J9
+U 1 1 6181E3FA
+P 3900 3650
+F 0 "J9" H 3818 3325 50  0000 C CNN
+F 1 "Screw_Terminal_01x02" H 3818 3416 50  0000 C CNN
+F 2 "TerminalBlock_Phoenix:TerminalBlock_Phoenix_MKDS-3-2-5.08_1x02_P5.08mm_Horizontal" H 3900 3650 50  0001 C CNN
+F 3 "~" H 3900 3650 50  0001 C CNN
+	1    3900 3650
+	-1   0    0    1
+$EndComp
+Wire Wire Line
+	4200 3650 4200 3800
+Wire Wire Line
+	4200 3400 4200 3550
 $EndSCHEMATC
