File: playboard.kicad_pcb (KiCad board)
At the start: 2 copper layers, 96 parts, among them J1 Conn_ARM_JTAG_SWD_10, J2 USB_B_Micro, J3 Conn_01x04_Male, J4 Conn_01x04_Male, J5 Conn_01x04_Male, J6 Conn_01x04_Male, J7 Conn_01x04_Male, J8 Conn_01x04_Male, Q1 AO3401A, Q2 FDV305N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

Commit message: update
Parts:
- removed C18: 10u, Capacitor_SMD:C_0402_1005Metric
- removed the D4 at (98.3, -14.7)
- removed the D4 at (100.9, 25.6)
- removed R8: 47, Resistor_SMD:R_0402_1005Metric
- removed Y2: 32.768 kHz, Crystal:Crystal_SMD_0603-4Pin_6.0x3.5mm
- added ABM8-20.000MHZ-B2-T1: 20MHz, Crystal:Crystal_SMD_0603-4Pin_6.0x3.5mm, F.Cu at (62.5, 59.0)
- added D4: ASMB-KTF0-0A306, ASMB-KTF0-0A306:LED_ASMB-KTF0-0A306, F.Cu at (68.8, 84.0)
- added D7: D_Schottky_Small, Diode_SMD:D_0603_1608Metric, F.Cu at (83.3, 81.9)
- added D8: D_Schottky_Small, Diode_SMD:D_0603_1608Metric, F.Cu at (83.7, 84.0)
- added J9: Screw_Terminal_01x02, TerminalBlock_Phoenix:TerminalBlock_Phoenix_MKDS-3-2-5.08_1x02_P5.08mm_Horizontal, F.Cu at (97.5, 72.5)
- C11: value 10u -> 47u
- C13: value 10u -> 220u; footprint Capacitor_SMD:C_0805_2012Metric -> Capacitor_SMD:CP_Elec_5x3
- C16, C17: value 12p -> 9pF
- F1: value Polyfuse_Small -> 500mA
- J2: value USB_B_Micro -> 47346-0001
- L1: value L_Small -> 27u; footprint Inductor_SMD:L_0603_1608Metric -> Inductor_SMD:L_7.3x7.3_H4.5
- R6: value 1k -> 3k
- R7: value 1k -> 1k78
- U1: value STM32F446RETx -> STM32F411RETx
- U2: value LMR33620ADDA -> MIC4684; footprint Package_SO:Texas_HSOP-8-1EP_3.9x4.9mm_P1.27mm_ThermalVias -> Package_SO:SOIC-8_3.9x4.9mm_P1.27mm
- U5: value HTS221 -> SHT30-DIS; footprint HTS221:XDCR_HTS221 -> Sensor_Humidity:Sensirion_DFN-8-1EP_2.5x2.5mm_P0.5mm_EP1.1x1.7mm
- Y1: value 16MHz -> ABS06-32.768KHZ-T; footprint Crystal:Crystal_SMD_0603-4Pin_6.0x3.5mm -> ABS06-32:XTAL_ABS06-32.768KHZ-T
- moved D2 120.6 mm to (49.5, 98.2)
- moved R21 114.5 mm to (42.8, 78.2)
- moved C26 110.5 mm to (45.2, 78.0)
- moved D3 104.2 mm to (87.1, 89.0)
- moved F1 102.1 mm to (51.6, 95.5)
- moved U5 101.0 mm to (45.3, 75.0)
- moved R20 100.9 mm to (60.8, 74.2)
- moved Q1 97.8 mm to (48.5, 93.8)
- moved R6 95.6 mm to (83.0, 87.1)
- moved C28 95.0 mm to (86.5, 44.0), turned to 270 degrees
- moved D5 95.0 mm to (70.1, 101.9)
- moved C24 93.5 mm to (67.2, 76.1)
- moved U4 93.2 mm to (63.6, 75.0)
- moved C11 93.0 mm to (78.7, 81.6)
- moved R7 92.7 mm to (86.7, 77.9)
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Connections:
- C13 pad 1: Net-(C13-Pad1) -> +3V3
- C14 pad 1: Net-(C14-Pad1) -> Net-(ABM8-20.000MHZ-B2-T1-Pad3)
- C17 pad 1: Net-(C17-Pad1) -> OSC32_OUT
- J2 pad S1: (no net) -> Net-(J2-PadS1)
- J2 pad S2: (no net) -> Net-(J2-PadS1)
- J2 pad S3: (no net) -> Net-(J2-PadS1)
- J2 pad S4: (no net) -> Net-(J2-PadS1)
- J2 pad S5: (no net) -> Net-(J2-PadS1)
- J2 pad S6: (no net) -> Net-(J2-PadS1)
- R5 pad 1: Net-(C14-Pad1) -> Net-(ABM8-20.000MHZ-B2-T1-Pad3)
- R6 pad 1: GND -> Net-(R6-Pad1)
- R6 pad 2: Net-(R6-Pad2) -> +3V3
- R7 pad 1: Net-(R6-Pad2) -> GND
- R7 pad 2: +3V3 -> Net-(R6-Pad1)
- U2 pad 1: GND -> Net-(C15-Pad2)
- U2 pad 2: Net-(C11-Pad1) -> GND
- U2 pad 4: Net-(U2-Pad4) -> Net-(C15-Pad1)
- U2 pad 5: Net-(R6-Pad2) -> Net-(R6-Pad1)
- U2 pad 6: Net-(C13-Pad1) -> GND
- U2 pad 7: Net-(C15-Pad1) -> GND
- U2 pad 8: Net-(C15-Pad2) -> Net-(C11-Pad1)
- U5 pad 1: +3V3 -> Net-(U5-Pad1)
- U5 pad 2: TEMP_SCL -> Net-(U5-Pad2)
- U5 pad 3: TEMP_DATARDY -> Net-(U5-Pad3)
- U5 pad 4: TEMP_SDA -> Net-(U5-Pad4)
- U5 pad 5: GND -> Net-(U5-Pad5)
- U5 pad 6: TEMP_CS -> Net-(U5-Pad6)
- Y1 pad 1: HSE_IN -> OSC32_IN
- Y1 pad 2: GND -> OSC32_OUT
Other:
- board outline added: 61.5 x 70 mm
