File: playboard.sch (KiCad schematic (older format))
At the start: 40 parts, among them Q1 AO3401A, SW1 SW_SPDT, U1 STM32F446RETx, U2 LMR33620ADDA, Y1 16MHz, Y2 32.768 kHz

Commit message: update
Parts:
- removed C13: 10u, Capacitor_SMD:C_0805_2012Metric, symbol Device:C_Small
- removed C18: 10u, Capacitor_SMD:C_0402_1005Metric, symbol Device:C_Small
- removed R6, R7, R9: 1k, Resistor_SMD:R_0402_1005Metric, symbol Device:R_Small
- removed R8: 47, Resistor_SMD:R_0402_1005Metric, symbol Device:R_Small_US
- removed U1: STM32F446RETx, Package_QFP:LQFP-64_10x10mm_P0.5mm, symbol MCU_ST_STM32F4:STM32F446RETx
- removed U2: LMR33620ADDA, Package_SO:Texas_HSOP-8-1EP_3.9x4.9mm_P1.27mm_ThermalVias, symbol Regulator_Switching:LMR33620ADDA
- removed Y2: 32.768 kHz, Crystal:Crystal_SMD_0603-4Pin_6.0x3.5mm, symbol Device:Crystal_GND24_Small
- added C13: 220u, Capacitor_SMD:CP_Elec_5x3, symbol Device:CP_Small
- added D7, D8: D_Schottky_Small, Diode_SMD:D_0603_1608Metric, symbol Device:D_Schottky_Small
- added R6: 3k, Resistor_SMD:R_0402_1005Metric, symbol Device:R_Small_US
- added R7: 1k78, Resistor_SMD:R_0402_1005Metric, symbol Device:R_Small_US
- added R9: 1k, Resistor_SMD:R_0402_1005Metric, symbol Device:R_Small_US
- added U1: STM32F411RETx, Package_QFP:LQFP-64_10x10mm_P0.5mm, symbol MCU_ST_STM32F4:STM32F411RETx
- added U2: MIC4684, Package_SO:SOIC-8_3.9x4.9mm_P1.27mm, symbol Regulator_Switching:MIC4684
- added Y1: ABS06-32.768KHZ-T, ABS06-32:XTAL_ABS06-32.768KHZ-T, symbol ABS06-32.768KHZ-T:ABS06-32.768KHZ-T
- ABM8-20.000MHZ-B2-T1: renamed from Y1; value 16MHz -> 20MHz
- C11: value 10u -> 47u
- C16, C17: value 12p -> 9pF
- L1: value L_Small -> 27u; footprint Inductor_SMD:L_0603_1608Metric -> Inductor_SMD:L_7.3x7.3_H4.5
Connections:
- net +3.3VA: now also U1.13 (VDDA)
- net +3V3: now also C13.1, R6.2, U1.1 (VBAT), U1.19 (VDD), U1.32 (VDD), U1.48 (VDD), U1.64 (VDD)
- net ACC_CS!: now also U1.24 (PC4)
- net ACC_INT1: now also U1.27 (PB1)
- net ACC_INT2: now also U1.28 (PB2)
- net ACC_MISO_SA0: now also U1.22 (PA6)
- net ACC_MOSI_SDA: now also U1.23 (PA7)
- net ACC_SCLK_SCL: now also U1.21 (PA5)
- net ADC1_IN1: now also U1.15 (PA1)
- net BOOT0: now also U1.60 (BOOT0)
- net BUTTON_1: now also U1.26 (PB0)
- net BUTTON_2: now also U1.25 (PC5)
- net DAC_OUT1: now also U1.20 (PA4)
- net EXT_GPIO_PC0: now also U1.8 (PC0)
- net EXT_GPIO_PC3: now also U1.11 (PC3)
- net FLASH_CS!: now also U1.33 (PB12)
- net FLASH_HOLD!: now also U1.40 (PC9)
- net FLASH_MISO: now also U1.35 (PB14)
- net FLASH_MOSI: now also U1.36 (PB15)
- net FLASH_SCLK: now also U1.34 (PB13)
- net FLASH_WP!: now also U1.42 (PA9)
- net GND: now also C13.2, D8.2 (A), R7.1, R9.1, U1.12 (VSSA), U1.18 (VSS), U1.31 (VSS), U1.47 (VSS), U1.63 (VSS), U2.2 (GND), U2.6 (GND), U2.7 (GND)
- net HSE_IN: now also U1.5 (PH0)
- net HSE_OUT: now also U1.6 (PH1)
- net MCO_1: now also U1.41 (PA8)
- net MIC_MODE: now also U1.9 (PC1)
- net MIC_VOUT_ANALOG: now also U1.10 (PC2)
- net NRST: now also U1.7 (NRST)
- net OSC32_IN: now also U1.3 (PC14), Y1.1
- net OSC32_OUT: now also C17.1, U1.4 (PC15), Y1.2
- net RGB_BLUE: now also U1.39 (PC8)
- net RGB_GREEN: now also U1.38 (PC7)
- net RGB_RED: now also U1.37 (PC6)
- net SPI3_MISO: now also U1.52 (PC11)
- net SPI3_MOSI: now also U1.53 (PC12)
- net SPI3_SCLK: now also U1.51 (PC10)
- net SWCLK: now also U1.49 (PA14)
- net SWDIO: now also U1.46 (PA13)
- net SWO: now also U1.55 (PB3)
- net TEMP_CS: now also U1.56 (PB4)
- net TEMP_DATARDY: now also U1.57 (PB5)
- net TEMP_SCL: now also U1.61 (PB8)
- net TEMP_SDA: now also U1.59 (PB7)
- net TIM11_CH1: now also U1.62 (PB9)
- net TIM5_CH1: now also U1.14 (PA0)
- net USART1_RX: now also U1.43 (PA10)
- net USART1_TX: now also U1.58 (PB6)
- net USART2_RX: now also U1.17 (PA3)
- net USART2_TX: now also U1.16 (PA2)
- net USB_D+: now also U1.45 (PA12)
- net USB_D-: now also U1.44 (PA11)
- net USER_LD1: now also U1.29 (PB10)
- net USER_LD2: now also U1.50 (PA15)
- net WOS_TRIGGER: now also U1.2 (PC13)
- net at C4.1: now also U1.30 (VCAP1)
- net at C11.1, FB2.2: now also D7.2 (A), U2.3 (VIN), U2.8 (EN)
- net at C15.1: now also D7.1 (K), U2.4 (BS)
- net at C15.2, L1.1: now also D8.1 (K), U2.1 (SW)
- net at D3.1 (K): now also R9.2
- new net: R6.1, R7.2, U2.5 (FB)
- no-connect marks 2 -> 1
Other:
- moved on the sheet: C15, L1
